File: efuse.kicad_sch (KiCad schematic)
At the start: 0 parts

Commit message: schem: add TPS259472A efuse
Parts:
- added C1: C, Capacitor_SMD:C_0402_1005Metric, symbol Device:C
- added C2: 1n, Capacitor_SMD:C_0402_1005Metric, symbol Device:C
- added C4: 1u, Capacitor_SMD:C_0402_1005Metric, symbol Device:C
- added D13: GREEN, LED_SMD:LED_0805_2012Metric, symbol Device:LED
- added R10, R3: 10k, Resistor_SMD:R_0402_1005Metric, symbol Device:R
- added R11, R12, R13: 1k5, Resistor_SMD:R_0402_1005Metric, symbol Device:R
- added R14, R4: 5k1, Resistor_SMD:R_0402_1005Metric, symbol Device:R
- added R5: 390k, Resistor_SMD:R_0402_1005Metric, symbol Device:R
- added U1: TPS259472A, symbol GLCS:TPS259472x
Connections:
- new net: R12.1, R13.1, R14.1, U1.9 (ILM)
- new net: C2.1, U1.7 (DVDT)
- new net: R5.1, U1.2 (OVCSEL)
- new net: C1.1, U1.10 (ITIMER)
- new net: R10.1, R11.2, U1.4 (PGTH)
- new net +3V3: R3.2, R4.1
- new net EN: R3.1, U1.1 (EN/UVLO)
- new net GND: C1.2, C2.2, C4.1, D13.1 (K), R11.1, R12.2, R13.2, R14.2, R5.2, U1.8 (GND)
- new net IN: C4.2, U1.5 (IN)
- new net OUT: R10.2, U1.6 (OUT)
- new net PG: D13.2 (A), R4.2, U1.3 (PG)
Other:
- note added: "Slew Rate 2A limit for 500uF load -> 4V/ms -> Cdvdt = 500pF (BOM consolidation) For 1n -> SR = 2V/ms Ilim Req=653.85Ω ->Ilim=5.1A ->I=Vilm(µV)/(180*650)"
