File: power.kicad_sch (KiCad schematic)
At the start: 9 parts, among them U6 TPS5430DDA

Commit message: schem: add efuse page
Other:
- added sheet Efuse (efuse.kicad_sch)
- moved on the sheet: C25, C27, C30, C31, D7, L6, R21, R22, U6

Commit message: schem: add TPS259472A efuse
Other:
- sheet Efuse ports: added EN, IN, OUT, PG; removed none
Changed lines of the file:
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@@
 	(sheet
 		(at 134.62 39.37)
-		(size 12.7 13.97)
+		(size 12.7 7.62)
 		(exclude_from_sim no)
 		(in_bom yes)
@@
 		)
 		(property "Sheetfile" "efuse.kicad_sch"
-			(at 134.62 53.9246 0)
+			(at 134.62 47.5746 0)
 			(effects
 				(font
@@
 				)
 				(justify left top)
+				(hide yes)
 			)
 		)
+		(pin "EN" input
+			(at 134.62 44.45 180)
+			(effects
+				(font
+					(size 1.27 1.27)
+				)
+				(justify left)
+			)
+		)
+		(pin "PG" output
+			(at 147.32 44.45 0)
+			(effects
+				(font
+					(size 1.27 1.27)
+				)
+				(justify right)
+			)
+		)
+		(pin "OUT" input
+			(at 147.32 40.64 0)
+			(effects
+				(font
+					(size 1.27 1.27)
+				)
+				(justify right)
+			)
+		)
+		(pin "IN" input
+			(at 134.62 40.64 180)
+			(effects
+				(font
+					(size 1.27 1.27)
+				)
+				(justify left)
+			)
+		)

Commit message: schem: add TPS56A37 12V SMPS
Parts:
- added BT1: 18v, symbol Device:Battery
- added C26, C28: 10u, Capacitor_SMD:C_0805_2012Metric, symbol Device:C
- added C29, C32: 0u1, Capacitor_SMD:C_0402_1005Metric, symbol Device:C
- added C33: 47p, Capacitor_SMD:C_0402_1005Metric, symbol Device:C
- added C34, C35, C8, C9: 22u, Capacitor_SMD:C_0805_2012Metric, symbol Device:C
- added D8: RED, LED_SMD:LED_0603_1608Metric, symbol Device:LED
- added L7: 5u6, Inductor_SMD:L_10.4x10.4_H4.8, symbol Device:L
- added NT1: NetTie_2, NetTie:NetTie-2_SMD_Pad0.5mm, symbol Device:NetTie_2
- added R15: 52k3, Resistor_SMD:R_0402_1005Metric, symbol Device:R
- added R18, R25: 5k1, Resistor_SMD:R_0402_1005Metric, symbol Device:R
- added R28: 100k, Resistor_SMD:R_0402_1005Metric, symbol Device:R
- added U7: TPS56A37, GLCS:Texas_RPA0010A_VQFN-HR-10_3x3mm_P0.5mm, symbol GLCS:TPS56A37
Connections:
- net GND: now also BT1.2 (-), C26.2, C28.2, C29.2, C34.2, C35.2, C8.2, C9.2, D8.1 (K), NT1.2, U7.9 (PGND)
- net +Vin: no longer names the net of C25.1, U6.5 (EN), U6.7 (VIN)
- net +Vin: now also BT1.1 (+), C26.1, C28.1, C29.1, U7.8 (VIN)
- new net: C33.1, R25.1, R28.1, U7.2 (FB)
- new net: C32.1, U7.7 (BOOT)
- new net: C32.2, L7.1, U7.6 (SW)
- new net: R15.2, U7.10 (MODE)
- new net +12V: C33.2, C34.1, C35.1, C8.1, C9.1, L7.2, R18.1, R28.2
- new net AGND: NT1.1, R15.1, R25.2, U7.3 (AGND)
- new net PG_12V: D8.2 (A), R18.2, U7.4 (PG)
- no-connect marks 0 -> 2
Other:
- note added: "TPS56A37 12V"
- moved on the sheet: C25, C27, C30, C31, D7, L6, R21, R22, U6

Commit message: schem: add TPS56A37 5V SMPS
Parts:
- added C10, C11: 10u, Capacitor_SMD:C_0805_2012Metric, symbol Device:C
- added C12, C13: 0u1, Capacitor_SMD:C_0402_1005Metric, symbol Device:C
- added C14: 47p, Capacitor_SMD:C_0402_1005Metric, symbol Device:C
- added C15, C16, C17, C18: 22u, Capacitor_SMD:C_0805_2012Metric, symbol Device:C
- added D1: RED, LED_SMD:LED_0603_1608Metric, symbol Device:LED
- added L1: 5u6, Inductor_SMD:L_10.4x10.4_H4.8, symbol Device:L
- added NT2: NetTie_2, NetTie:NetTie-2_SMD_Pad0.5mm, symbol Device:NetTie_2
- added R16: 5k1, Resistor_SMD:R_0402_1005Metric, symbol Device:R
- added R17: 52k3, Resistor_SMD:R_0402_1005Metric, symbol Device:R
- added R19: 10k, Resistor_SMD:R_0402_1005Metric, symbol Device:R
- added R20: 73k2, Resistor_SMD:R_0402_1005Metric, symbol Device:R
- added U2: TPS56A37, GLCS:Texas_RPA0010A_VQFN-HR-10_3x3mm_P0.5mm, symbol GLCS:TPS56A37
Connections:
- net +12V: now also R16.1
- net GND: now also C10.2, C11.2, C12.2, C15.2, C16.2, C17.2, C18.2, D1.1 (K), NT2.2, U2.9 (PGND)
- net at BT1.1 (+), C25.1, C26.1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: now also C10.1, C11.1, C12.1, U2.8 (VIN)
- new net: C14.1, R19.2, R20.1, U2.2 (FB)
- new net: C13.2, L1.1, U2.6 (SW)
- new net: R17.2, U2.10 (MODE)
- new net: C13.1, U2.7 (BOOT)
- new net +5V: C14.2, C15.1, C16.1, C17.1, C18.1, L1.2, R20.2
- new net AGND2: NT2.1, R17.1, R19.1, U2.3 (AGND)
- new net PG_5V: D1.2 (A), R16.2, U2.4 (PG)
- no-connect marks 2 -> 4
Other:
- note added: "TPS56A37 5V"
- moved on the sheet: BT1, C25, C26, C27, C28, C29, C30, C31, C32, C33, C34, C35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

Commit message: schem: add battery esd tvs diode
Parts:
- added D2: D_TVS, Diode_SMD:D_SMA, symbol Device:D_TVS
Connections:
- net GND: now also D2.1 (A1)
- net at BT1.1 (+), C10.1, C11.1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: now also D2.2 (A2)
Other:
- moved on the sheet: BT1
Changed lines of the file:
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@@
 	)
 	(junction
+		(at 38.1 62.23)
+		(diameter 0)
+		(color 0 0 0 0)
+	)
+	(junction
 		(at 146.05 50.8)
 		(diameter 0)
@@
 	(wire
 		(pts
+			(xy 38.1 62.23) (xy 49.53 62.23)
+		)
+		(stroke
+			(width 0)
+			(type default)
+		)
+	)
+	(wire
+		(pts
 			(xy 25.4 40.64) (xy 67.31 40.64)
 		)
@@
 	(wire
 		(pts
-			(xy 25.4 68.58) (xy 25.4 62.23)
+			(xy 25.4 63.5) (xy 25.4 62.23)
 		)
 		(stroke
@@
 	(wire
 		(pts
-			(xy 25.4 62.23) (xy 49.53 62.23)
+			(xy 25.4 62.23) (xy 38.1 62.23)
 		)
 		(stroke
@@
 	(wire
 		(pts
-			(xy 25.4 78.74) (xy 25.4 80.01)
+			(xy 25.4 73.66) (xy 25.4 74.93)
 		)
 		(stroke
@@
 	(wire
 		(pts
+			(xy 38.1 72.39) (xy 38.1 74.93)
+		)
+		(stroke
+			(width 0)
+			(type default)
+		)
+	)
+	(wire
+		(pts
 			(xy 161.29 139.7) (xy 161.29 138.43)
 		)
@@
 	(wire
 		(pts
+			(xy 38.1 62.23) (xy 38.1 64.77)
+		)
+		(stroke
+			(width 0)
+			(type default)
+		)
+	)
+	(wire
+		(pts
 			(xy 60.96 129.54) (xy 71.12 129.54)
 		)
@@
 	(symbol
 		(lib_id "Device:Battery")
-		(at 25.4 73.66 0)
+		(at 25.4 68.58 0)
 		(unit 1)
 		(exclude_from_sim no)
@@
 		(fields_autoplaced yes)
 		(property "Reference" "BT1"
-			(at 29.21 71.8184 0)
+			(at 29.21 66.7384 0)
 			(effects
 				(font
@@
 		)
 		(property "Value" "18v"
-			(at 29.21 74.3584 0)
+			(at 29.21 69.2784 0)
 			(effects
 				(font
@@
 		)
 		(property "Footprint" ""
-			(at 25.4 72.136 90)
+			(at 25.4 67.056 90)
 			(effects
 				(font
@@
 		)
 		(property "Datasheet" "~"
-			(at 25.4 72.136 90)
+			(at 25.4 67.056 90)
 			(effects
 				(font
@@
 		)
 		(property "Description" "Multiple-cell battery"
-			(at 25.4 73.66 0)
+			(at 25.4 68.58 0)
 			(effects
 				(font
@@
 		)
 		(property "Sim.Device" "V"
-			(at 25.4 73.66 0)
+			(at 25.4 68.58 0)
 			(effects
 				(font
@@
 		)
 		(property "Sim.Type" "DC"
-			(at 25.4 73.66 0)
+			(at 25.4 68.58 0)
 			(effects
 				(font
@@
 		)
 		(property "Sim.Pins" "1=+ 2=-"
-			(at 25.4 73.66 0)
+			(at 25.4 68.58 0)
 			(effects
 				(font
@@
 	)
 	(symbol
+		(lib_id "Device:D_TVS")
+		(at 38.1 68.58 90)
+		(unit 1)
+		(exclude_from_sim no)
+		(in_bom yes)
+		(on_board yes)
+		(dnp no)
+		(fields_autoplaced yes)
+		(property "Reference" "D2"
+			(at 40.64 68.5799 90)
+			(effects
+				(font
+					(size 1.27 1.27)
+				)
+				(justify right)
+			)
+		)
+		(property "Value" "D_TVS"
+			(at 40.64 69.8499 90)
+			(effects
+				(font
+					(size 1.27 1.27)
+				)
+				(justify right)
+				(hide yes)
+			)
+		)
+		(property "Footprint" "Diode_SMD:D_SMA"
+			(at 38.1 68.58 0)
+			(effects
+				(font
+					(size 1.27 1.27)
+				)
+				(hide yes)
+			)
+		)
+		(property "Datasheet" "~"
+			(at 38.1 68.58 0)
+			(effects
+				(font
+					(size 1.27 1.27)
+				)
+				(hide yes)
+			)
+		)
+		(property "Description" "Bidirectional transient-voltage-suppression diode"
+			(at 38.1 68.58 0)
+			(effects
+				(font
+					(size 1.27 1.27)
+				)
+				(hide yes)
+			)
+		)
+		(property "Basic" "E"
+			(at 38.1 68.58 90)
+			(effects
+				(font
+					(size 1.27 1.27)
+				)
+				(hide yes)
+			)
+		)
+		(property "JLCPCB Part #" "C19077549"
+			(at 38.1 68.58 90)
+			(effects
+				(font
+					(size 1.27 1.27)
+				)
+				(hide yes)
+			)
+		)
+		(property "Manufacturer" "hongjiacheng"
+			(at 38.1 68.58 90)
+			(effects
+				(font
+					(size 1.27 1.27)
+				)
+				(hide yes)
+			)
+		)
+		(property "Manufacturer Part Number" "SMAJ33CA"
+			(at 38.1 68.58 90)
+			(effects
+				(font
+					(size 1.27 1.27)
+				)
+				(hide yes)
+			)
+		)
+		(pin "1"
+		)
+		(pin "2"
+		)
+		(instances
+			(project ""
+				(path "/8d7b287d-627f-46aa-8c27-0b5ed29ab4a2/0cc01053-a223-4e8e-b0aa-a1ec618db290"
+					(reference "D2")
+					(unit 1)
+				)
+			)
+		)
+	)
+	(symbol
 		(lib_id "Device:C")
 		(at 81.28 134.62 0)
@@
 	(symbol
 		(lib_id "power:GND")
-		(at 25.4 80.01 0)
+		(at 25.4 74.93 0)
 		(unit 1)
 		(exclude_from_sim no)
@@
 		(dnp no)
 		(property "Reference" "#PWR015"
-			(at 25.4 86.36 0)
+			(at 25.4 81.28 0)
 			(effects
 				(font
@@
 		)
 		(property "Value" "GND"
-			(at 29.464 81.534 0)
+			(at 29.464 76.454 0)
 			(effects
 				(font
@@
 		)
 		(property "Footprint" ""
-			(at 25.4 80.01 0)
+			(at 25.4 74.93 0)
 			(effects
 				(font
@@
 		)
 		(property "Datasheet" ""
-			(at 25.4 80.01 0)
+			(at 25.4 74.93 0)
 			(effects
 				(font
@@
 		)
 		(property "Description" "Power symbol creates a global label with name \"GND\" , ground"
-			(at 25.4 80.01 0)
+			(at 25.4 74.93 0)
 			(effects
 				(font
@@
 					(unit 1)
 				)
+			)
+		)
+	)
+	(symbol
+		(lib_id "power:GND")
+		(at 38.1 74.93 0)
+		(unit 1)
+		(exclude_from_sim no)
+		(in_bom yes)
+		(on_board yes)
+		(dnp no)
+		(property "Reference" "#PWR036"
+			(at 38.1 81.28 0)
+			(effects
+				(font
+					(size 1.27 1.27)
+				)
+				(hide yes)
+			)
+		)
+		(property "Value" "GND"
+			(at 42.164 76.454 0)
+			(effects
+				(font
+					(size 1.27 1.27)
+				)
+				(hide yes)
+			)
+		)
+		(property "Footprint" ""
+			(at 38.1 74.93 0)
+			(effects
+				(font
+					(size 1.27 1.27)
+				)
+				(hide yes)
+			)
+		)
+		(property "Datasheet" ""
+			(at 38.1 74.93 0)
+			(effects
+				(font
+					(size 1.27 1.27)
+				)
+				(hide yes)
+			)
+		)
+		(property "Description" "Power symbol creates a global label with name \"GND\" , ground"
+			(at 38.1 74.93 0)
+			(effects
+				(font
+					(size 1.27 1.27)
+				)
+				(hide yes)
+			)
+		)
+		(pin "1"
+		)
+		(instances
+			(project "valrob-carte-alim-cdf-1"
+				(path "/8d7b287d-627f-46aa-8c27-0b5ed29ab4a2/0cc01053-a223-4e8e-b0aa-a1ec618db290"
+					(reference "#PWR036")
+					(unit 1)
+				)

Commit message: schem: add TPS259472A 5V 5A efuse
Other:
- sheet Efuse renamed Efuse 12V 5A
- added sheet Efuse 5V 5A (efuse-5-5.kicad_sch)
- sheet Efuse 12V 5A: file efuse.kicad_sch -> efuse-12-5.kicad_sch
Changed lines of the file:
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@@
 	(wire
 		(pts
+			(xy 176.53 46.99) (xy 176.53 57.15)
+		)
+		(stroke
+			(width 0)
+			(type default)
+		)
+	)
+	(wire
+		(pts
 			(xy 92.71 95.25) (xy 101.6 95.25)
 		)
@@
 			(color 0 0 0 0.0000)
 		)
-		(property "Sheetname" "Efuse"
+		(property "Sheetname" "Efuse 12V 5A"
 			(at 125.73 15.7984 0)
 			(effects
@@
 			)
 		)
-		(property "Sheetfile" "efuse.kicad_sch"
+		(property "Sheetfile" "efuse-12-5.kicad_sch"
 			(at 125.73 23.4446 0)
 			(effects
@@
 				)
 			)
+		)
+	)
+	(sheet
+		(at 146.05 16.51)
+		(size 12.7 6.35)
+		(exclude_from_sim no)
+		(in_bom yes)
+		(on_board yes)
+		(dnp no)
+		(fields_autoplaced yes)
+		(stroke
+			(width 0.1524)
+			(type solid)
+		)
+		(fill
+			(color 0 0 0 0.0000)
+		)
+		(property "Sheetname" "Efuse 5V 5A"
+			(at 146.05 15.7984 0)
+			(effects
+				(font
+					(size 1.27 1.27)
+				)
+				(justify left bottom)
+			)
+		)
+		(property "Sheetfile" "efuse-5-5.kicad_sch"
+			(at 146.05 23.4446 0)
+			(effects
+				(font
+					(size 1.27 1.27)
+				)
+				(justify left top)
+				(hide yes)
+			)
+		)
+		(pin "EN" input
+			(at 146.05 21.59 180)
+			(effects
+				(font
+					(size 1.27 1.27)
+				)
+				(justify left)
+			)
+		)
+		(pin "PG" output
+			(at 158.75 21.59 0)
+			(effects
+				(font
+					(size 1.27 1.27)
+				)
+				(justify right)
+			)
+		)
+		(pin "OUT" input
+			(at 158.75 17.78 0)
+			(effects
+				(font
+					(size 1.27 1.27)
+				)
+				(justify right)
+			)
+		)
+		(pin "IN" input
+			(at 146.05 17.78 180)
+			(effects
+				(font
+					(size 1.27 1.27)
+				)
+				(justify left)
+			)
+		)
+		(instances
+			(project "valrob-carte-alim-cdf-1"
+				(path "/8d7b287d-627f-46aa-8c27-0b5ed29ab4a2/0cc01053-a223-4e8e-b0aa-a1ec618db290"
+					(page "4")
+				)
+			)
