File: efuse-12-5.kicad_sch (KiCad schematic)
At the start: 13 parts, among them U1 TPS259472A

Commit message: schem: add ILM pins and 12V 10A rail
Parts:
- U9: renamed from U1; Basic (none) -> X; JLCPCB Part # (none) -> C3662789; Manufacturer (none) -> Texas Instruments; Manufacturer Part Number (none) -> TPS259472ARPWR
- renumbered C4 to C39, C1 to C40, C2 to C41, D13 to D9, R3 to R46, R13 to R47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
Connections:
- net ILM: now reaches R47.1, R48.1, R49.1, U9.9 (ILM)
